File: LorRaAdapter.brd (EAGLE design)
At the start: 15.2 x 33.3 mm, 6 parts, among them P1 PINHD-2X4, U1 WIRELESS-LORA-RFM95W#SMD

Commit message: Add Midnight Fog logos
Parts:
- added LOGO1: MFDECLOGO_SQ_5MM, _my_logos:MFDEC_SQ_5MM
Changed lines of the file:
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@@
 <attribute name="VALUE" x="11.049" y="-1.651" size="1.27" layer="27"/>
 </element>
+<element name="LOGO1" library="_my_logos" package="MFDEC_SQ_5MM" value="MFDECLOGO_SQ_5MM" x="8.89" y="14.224" smashed="yes" rot="MR0"/>
 </elements>
 <signals>
