File: LorRaBaseBoard.brd (EAGLE design)
At the start: 30.5 x 26.3 mm, 6 parts, among them J4 U.FL, X1 BU-SMA-H

Commit message: Add Midnight Fog logos
Parts:
- added LOGO1: MFDECLOGO_SQ_8MM, _my_logos:MFDEC_SQ_8MM
Changed lines of the file:
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@@
 <wire x1="0" y1="26.34" x2="0" y2="0" width="0" layer="20"/>
 <text x="19.05" y="1.27" size="1.778" layer="21">v1.0</text>
-<text x="21.59" y="13.97" size="1.778" layer="22" rot="MR0">LoRaB v1.0</text>
+<text x="20.32" y="10.16" size="1.778" layer="22" rot="MR0">LoRaB v1.0</text>
 </plain>
 <attributes>
@@
 <attribute name="POPULARITY" value="4" x="13.97" y="5.08" size="1.778" layer="27" rot="R270" display="off"/>
 </element>
+<element name="LOGO1" library="_my_logos" package="MFDEC_SQ_8MM" value="MFDECLOGO_SQ_8MM" x="19.05" y="12.7" smashed="yes" rot="MR0"/>
 </elements>
 <signals>

Commit message: Renamed antenna connectors.
Parts:
- renumbered J4 to A2, X1 to A1
Changed lines of the file:
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@@
 <drawing>
 <settings>
-<setting alwaysvectorfont="yes"/>
+<setting alwaysvectorfont="no"/>
 <setting verticaltext="up"/>
 </settings>
@@
 <attribute name="VALUE" x="27.432" y="3.81" size="0.6096" layer="27" font="vector" ratio="20" rot="R90"/>
 </element>
-<element name="J4" library="SparkFun-Connectors" package="U.FL" value="U.FL" x="21.59" y="5.08" smashed="yes" rot="R90">
+<element name="A2" library="SparkFun-Connectors" package="U.FL" value="U.FL" x="21.59" y="5.08" smashed="yes" rot="R90">
 <attribute name="PROD_ID" value="CONN-09193" x="48.26" y="20.32" size="1.778" layer="27" rot="R90" display="off"/>
 <attribute name="SF_ID" value="WRL-09144" x="48.26" y="20.32" size="1.778" layer="27" rot="R90" display="off"/>
 </element>
 <element name="U$1" library="diy-modules" package="WIRELESS-LORA-RFM95W#SMD" value="WIRELESS-LORA-RFM95W#SMD" x="13.97" y="16.51" smashed="yes"/>
-<element name="X1" library="con-coax" library_urn="urn:adsk.eagle:library:133" package="BU-SMA-H" package3d_urn="urn:adsk.eagle:package:6206/1" value="BU-SMA-H" x="13.97" y="5.08" smashed="yes" rot="R270">
+<element name="A1" library="con-coax" library_urn="urn:adsk.eagle:library:133" package="BU-SMA-H" package3d_urn="urn:adsk.eagle:package:6206/1" value="BU-SMA-H" x="13.97" y="5.08" smashed="yes" rot="R270">
 <attribute name="MF" value="" x="13.97" y="5.08" size="1.778" layer="27" rot="R270" display="off"/>
 <attribute name="MPN" value="" x="13.97" y="5.08" size="1.778" layer="27" rot="R270" display="off"/>
@@
 <contactref element="U$1" pad="B7"/>
 <contactref element="J2" pad="2"/>
-<contactref element="J4" pad="1"/>
-<contactref element="J4" pad="2"/>
-<contactref element="X1" pad="3"/>
-<contactref element="X1" pad="2"/>
-<contactref element="X1" pad="5"/>
-<contactref element="X1" pad="4"/>
+<contactref element="A2" pad="1"/>
+<contactref element="A2" pad="2"/>
+<contactref element="A1" pad="3"/>
+<contactref element="A1" pad="2"/>
+<contactref element="A1" pad="5"/>
+<contactref element="A1" pad="4"/>
 <wire x1="24.93593125" y1="8.8392" x2="22.26513125" y2="11.51" width="0.254" layer="1"/>
 <wire x1="22.26513125" y1="11.51" x2="21.47" y2="11.51" width="0.254" layer="1"/>
@@
 <contactref element="U$1" pad="B8"/>
 <contactref element="J2" pad="1"/>
-<contactref element="J4" pad="FEED"/>
-<contactref element="X1" pad="1"/>
+<contactref element="A2" pad="FEED"/>
+<contactref element="A1" pad="1"/>
 <wire x1="21.59" y1="9.51" x2="21.47" y2="9.51" width="0.254" layer="1"/>
 <wire x1="13.97" y1="5.08" x2="17.02486875" y2="5.08" width="0.254" layer="1"/>
