File: LoRaBaseBoard.brd (EAGLE design)
At the start: 30.5 x 26.3 mm, 7 parts

Commit message: Fixed fill distance. Generated CAM files. Generated PNG preview.
Other:
- board text added: "LoRaB v1.1"
- board text added: "v1.1"
- board text removed: "LoRaB v1.0"
- board text removed: "v1.0"
Changed lines of the file:
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@@
 <drawing>
 <settings>
-<setting alwaysvectorfont="no"/>
+<setting alwaysvectorfont="yes"/>
 <setting verticaltext="up"/>
 </settings>
@@
 <wire x1="30.46" y1="26.34" x2="0" y2="26.34" width="0" layer="20"/>
 <wire x1="0" y1="26.34" x2="0" y2="0" width="0" layer="20"/>
-<text x="19.05" y="1.27" size="1.778" layer="21" font="vector">v1.0</text>
-<text x="20.32" y="10.16" size="1.778" layer="22" font="vector" rot="MR0">LoRaB v1.0</text>
+<text x="19.05" y="1.27" size="1.778" layer="21" font="vector">v1.1</text>
+<text x="20.32" y="10.16" size="1.778" layer="22" font="vector" rot="MR0">LoRaB v1.1</text>
 </plain>
 <attributes>
@@
 <wire x1="19.0698" y1="5.08" x2="20.215" y2="5.08" width="0.254" layer="1"/>
 <wire x1="20.215" y1="5.08" x2="21.59" y2="5.08" width="0.254" layer="1"/>
-<polygon width="0.254" layer="1" isolate="0.254">
+<polygon width="0.3048" layer="1" isolate="0.254">
 <vertex x="0" y="0"/>
 <vertex x="0" y="26.67"/>
@@
 <vertex x="30.48" y="0"/>
 </polygon>
-<polygon width="0.1524" layer="16" isolate="0.254">
+<polygon width="0.3048" layer="16" isolate="0.254">
 <vertex x="0" y="0"/>
 <vertex x="0" y="26.67"/>
